File: power.kicad_sch (KiCad schematic)
At the start: 19 parts, among them SW1 SW_DPDT_x2, T1 DST-5-36, U1 AP63205WU

Commit message: Common PSU
Parts:
- added F1: Polyfuse, symbol Device:Polyfuse
- TP2: value 5VDC -> 5VDCI
Connections:
- net +5V: now also F1.2; no longer C6.1, C7.1, L1.2, TP2.1, U1.1 (FB)
- new net +5VI2: C6.1, C7.1, F1.1, L1.2, TP2.1, U1.1 (FB)
