File: daughter/filtering.kicad_sch (KiCad schematic)
At the start: 4 parts

Commit message: Common PSU
Parts:
- renumbered C13 to C19, C12 to C20, L1 to L2
Changed lines of the file:
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@@
 		(on_board yes)
 		(dnp no)
-		(property "Reference" "L1"
+		(property "Reference" "L2"
 			(at 167.132 74.168 90)
 			(effects
@@
 			(project ""
 				(path "/9e050361-84ba-4b41-8bc1-d0f304e5538b/f2cc7818-958e-4ae3-9893-db5d97bb3573"
-					(reference "L1")
+					(reference "L2")
 					(unit 1)
 				)
@@
 		(on_board yes)
 		(dnp no)
-		(property "Reference" "C12"
+		(property "Reference" "C20"
 			(at 172.974 77.978 0)
 			(effects
@@
 			(project ""
 				(path "/9e050361-84ba-4b41-8bc1-d0f304e5538b/f2cc7818-958e-4ae3-9893-db5d97bb3573"
-					(reference "C12")
+					(reference "C20")
 					(unit 1)
 				)
@@
 		(on_board yes)
 		(dnp no)
-		(property "Reference" "C13"
+		(property "Reference" "C19"
 			(at 165.354 77.978 0)
 			(effects
@@
 			(project ""
 				(path "/9e050361-84ba-4b41-8bc1-d0f304e5538b/f2cc7818-958e-4ae3-9893-db5d97bb3573"
-					(reference "C13")
-					(unit 1)
-				)
+					(reference "C19")
+					(unit 1)
+				)
