File: daughter/usb.kicad_sch (KiCad schematic)
At the start: 13 parts, among them J1 USB_C_Receptacle_USB2.0_14P, U2 TLV1117-33

Commit message: Common PSU
Parts:
- renumbered C11 to C17, C10 to C18, F1 to F2, TP3 to TP10, TP6 to TP11, TP5 to TP12, TP4 to TP13, TP1 to TP8, TP2 to TP9
Other:
- moved on the sheet: C17, C18, U2
